File: simon/board/_autosave-simon.kicad_pcb (KiCad board)
At the start: 2 copper layers, 18 parts, among them IC1 ATTINY85-S, SW1 button, SW2 button, SW3 button, SW4 button, SW5 on/off

Commit message: added routing single layer
Parts:
- moved SW1 6.60 mm to (239.8, 94.0), turned to 180 degrees
Routing:
- net PB0: track 44.6 -> 57.5 mm
- net +3V3: track 90.9 -> 97.8 mm
- net GND: track 175.7 -> 178.1 mm
