File: simon/board/simon.kicad_pcb (KiCad board)
At the start: 2 copper layers, 18 parts, among them IC1 ATTINY85-S, SW1 button, SW2 button, SW3 button, SW4 button, SW5 on/off

Commit message: boad layout
Parts:
- BT1: moved to B.Cu
- IC1: footprint simon:SOIC8W -> Housings_DIP:DIP-8_W7.62mm_LongPads
- SW5: footprint Buttons_Switches_SMD:SW_SPST_FSMSM -> Connect:PINHEAD1-3
- moved BT1 118.6 mm to (138.4, 97.8)
- moved SW3 108.6 mm to (99.1, 76.2), turned to 270 degrees
- moved SP1 105.0 mm to (100.3, 123.2)
- moved D1 104.6 mm to (144.8, 81.3), turned to 0 degrees
- moved IC1 97.5 mm to (124.5, 95.2)
- moved SW2 94.3 mm to (124.5, 68.6)
- moved D2 93.7 mm to (127.0, 111.8)
- moved SW5 93.0 mm to (156.2, 111.8)
- moved R4 92.3 mm to (121.9, 88.9)
- moved D3 92.3 mm to (129.5, 55.9)
- moved R1 92.3 mm to (149.9, 99.1)
- moved R2 92.3 mm to (132.1, 88.9)
- moved R3 92.3 mm to (127.0, 78.7)
- moved R5 92.3 mm to (142.2, 109.2)
- moved R6 92.3 mm to (101.6, 91.4)
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Routing:
- net GND: track 175.7 -> 0.00 mm
- net PB2: track 96.7 -> 0.00 mm
- net +3V3: track 90.9 -> 0.00 mm
- net PB3: track 66.3 -> 0.00 mm
- net Net-(D1-Pad2): track 53.0 -> 0.00 mm
- net Net-(D3-Pad2): track 47.7 -> 0.00 mm
- net PB0: track 44.6 -> 0.00 mm
- net Net-(R2-Pad1): track 30.0 -> 0.00 mm
- net Net-(R4-Pad1): track 23.0 -> 0.00 mm
- net Net-(BT1-Pad1): track 17.0 -> 0.00 mm
- net PB4: track 15.0 -> 0.00 mm
- net Net-(R3-Pad1): track 14.2 -> 0.00 mm
- net PB1: track 9.35 -> 0.00 mm
Other:
- board outline added: 101.6 x 106.7 mm
